File: pca9535bowing.brd (EAGLE design)
At the start: 28.3 x 23.2 mm, 4 parts

Commit message: first layout
Parts:
- added RN1, RN2, RN3, RN4: 150, resistor-dil:CAY16
- added RN5, RN6, RN7, RN8: 100k, resistor-dil:CAY16
- moved PB_OUT 25.4 mm to (1.40, 21.7), turned to 0 degrees
Connections:
- removed net INT-: PA_OUT.3
- new net N$1: RN7.5, RN7.6, RN7.7, RN7.8, RN8.5, RN8.6, RN8.7, RN8.8
- new net N$10: PB_IN.8, RN2.4, RN7.1
- new net N$11: PA_IN.11, RN3.1, RN6.4
- new net N$12: PA_IN.10, RN3.2, RN6.3
- new net N$13: PA_IN.9, RN3.3, RN6.2
- new net N$14: PA_IN.8, RN3.4, RN6.1
- new net N$15: PA_IN.7, RN4.1, RN5.4
- new net N$16: PA_IN.6, RN4.2, RN5.3
- new net N$17: PA_IN.5, RN4.3, RN5.2
- new net N$18: PA_IN.4, RN4.4, RN5.1
- new net N$19: PA_IN.1, PA_OUT.1
- new net N$2: RN5.5, RN5.6, RN5.7, RN5.8, RN6.5, RN6.6, RN6.7, RN6.8
- new net N$20: PA_IN.2, PA_OUT.2
- new net N$21: PA_IN.3, PA_OUT.3
- new net N$22: PA_OUT.4, RN4.5
- new net N$23: PA_OUT.5, RN4.6
- new net N$24: PA_OUT.6, RN4.7
- new net N$25: PA_OUT.7, RN4.8
- new net N$26: PA_OUT.8, RN3.5
- new net N$27: PA_OUT.9, RN3.6
- new net N$28: PA_OUT.10, RN3.7
- new net N$29: PA_OUT.11, RN3.8
- new net N$3: PB_IN.1, RN1.1, RN8.4
- new net N$30: PB_IN.11, PB_OUT.11
- new net N$31: PB_IN.10, PB_OUT.10
- new net N$32: PB_IN.9, PB_OUT.9
- new net N$33: PB_OUT.1, RN1.8
- new net N$34: PB_OUT.2, RN1.7
- new net N$35: PB_OUT.3, RN1.6
- new net N$36: PB_OUT.4, RN1.5
- new net N$37: PB_OUT.5, RN2.8
- new net N$38: PB_OUT.6, RN2.7
- new net N$39: PB_OUT.7, RN2.6
- new net N$4: PB_IN.2, RN1.2, RN8.3
- new net N$40: PB_OUT.8, RN2.5
- new net N$5: PB_IN.3, RN1.3, RN8.2
- new net N$6: PB_IN.4, RN1.4, RN8.1
- new net N$7: PB_IN.5, RN2.1, RN7.4
- new net N$8: PB_IN.6, RN2.2, RN7.3
- new net N$9: PB_IN.7, RN2.3, RN7.2

Commit message: forgot to connect the pull-ups to voltage...
Connections:
- removed net N$1: RN7.5, RN7.6, RN7.7, RN7.8, RN8.5, RN8.6, RN8.7, RN8.8
- removed net N$2: RN5.5, RN5.6, RN5.7, RN5.8, RN6.5, RN6.6, RN6.7, RN6.8
- removed net N$20: PA_IN.2, PA_OUT.2
- new net 5V: PA_IN.2, PA_OUT.2, RN5.5, RN5.6, RN5.7, RN5.8, RN6.5, RN6.6, RN6.7, RN6.8, RN7.5, RN7.6, RN7.7, RN7.8, RN8.5, RN8.6, RN8.7, RN8.8

Commit message: autorouted
Parts:
- moved RN4 1.52 mm to (16.3, 9.91)
- moved RN3 1.02 mm to (24.1, 9.40)
- moved RN5 1.02 mm to (16.3, 13.0)
- moved RN6 1.02 mm to (24.1, 13.0)
- moved RN1 0.76 mm to (3.30, 13.5)
- moved RN2 0.76 mm to (11.4, 13.5)
- moved RN7 0.76 mm to (11.4, 9.91)
- moved RN8 0.76 mm to (3.30, 9.91)
Routing:
- net 5V: track 0.00 -> 34.6 mm
- net N$5: track 0.00 -> 14.6 mm
- net N$14: track 0.00 -> 11.8 mm
- net N$17: track 0.00 -> 11.6 mm, vias 0 -> 1
- net N$10: track 0.00 -> 11.6 mm
- net N$22: track 0.00 -> 11.6 mm, vias 0 -> 1
- net N$8: track 0.00 -> 11.5 mm, vias 0 -> 1
- net N$29: track 0.00 -> 11.4 mm, vias 0 -> 1
- net N$9: track 0.00 -> 11.2 mm, vias 0 -> 1
- net N$12: track 0.00 -> 11.2 mm, vias 0 -> 1
- net N$23: track 0.00 -> 11.1 mm, vias 0 -> 1
- net N$18: track 0.00 -> 11.1 mm, vias 0 -> 1
- net N$40: track 0.00 -> 11.0 mm
- net N$16: track 0.00 -> 10.5 mm
- net N$6: track 0.00 -> 10.3 mm, vias 0 -> 1
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