File: pca9535bowing.sch (EAGLE design)
At the start: 4 parts

Commit message: first layout
Parts:
- added RN1, RN2, RN3, RN4: 150, resistor-dil:4R-NCAY16
- added RN5, RN6, RN7, RN8: 100k, resistor-dil:4R-NCAY16
Connections:
- removed net INT-: PA_OUT.3
- new net N$1: RN7A.2, RN7B.2, RN7C.2, RN7D.2, RN8A.2, RN8B.2, RN8C.2, RN8D.2
- new net N$10: PB_IN.8, RN2D.1, RN7A.1
- new net N$11: PA_IN.11, RN3A.1, RN6D.1
- new net N$12: PA_IN.10, RN3B.1, RN6C.1
- new net N$13: PA_IN.9, RN3C.1, RN6B.1
- new net N$14: PA_IN.8, RN3D.1, RN6A.1
- new net N$15: PA_IN.7, RN4A.1, RN5D.1
- new net N$16: PA_IN.6, RN4B.1, RN5C.1
- new net N$17: PA_IN.5, RN4C.1, RN5B.1
- new net N$18: PA_IN.4, RN4D.1, RN5A.1
- new net N$19: PA_IN.1, PA_OUT.1
- new net N$2: RN5A.2, RN5B.2, RN5C.2, RN5D.2, RN6A.2, RN6B.2, RN6C.2, RN6D.2
- new net N$20: PA_IN.2, PA_OUT.2
- new net N$21: PA_IN.3, PA_OUT.3
- new net N$22: PA_OUT.4, RN4D.2
- new net N$23: PA_OUT.5, RN4C.2
- new net N$24: PA_OUT.6, RN4B.2
- new net N$25: PA_OUT.7, RN4A.2
- new net N$26: PA_OUT.8, RN3D.2
- new net N$27: PA_OUT.9, RN3C.2
- new net N$28: PA_OUT.10, RN3B.2
- new net N$29: PA_OUT.11, RN3A.2
- new net N$3: PB_IN.1, RN1A.1, RN8D.1
- new net N$30: PB_IN.11, PB_OUT.11
- new net N$31: PB_IN.10, PB_OUT.10
- new net N$32: PB_IN.9, PB_OUT.9
- new net N$33: PB_OUT.1, RN1A.2
- new net N$34: PB_OUT.2, RN1B.2
- new net N$35: PB_OUT.3, RN1C.2
- new net N$36: PB_OUT.4, RN1D.2
- new net N$37: PB_OUT.5, RN2A.2
- new net N$38: PB_OUT.6, RN2B.2
- new net N$39: PB_OUT.7, RN2C.2
- new net N$4: PB_IN.2, RN1B.1, RN8C.1
- new net N$40: PB_OUT.8, RN2D.2
- new net N$5: PB_IN.3, RN1C.1, RN8B.1
- new net N$6: PB_IN.4, RN1D.1, RN8A.1
- new net N$7: PB_IN.5, RN2A.1, RN7D.1
- new net N$8: PB_IN.6, RN2B.1, RN7C.1
- new net N$9: PB_IN.7, RN2C.1, RN7B.1
Other:
- moved on the sheet: PA_IN, PA_OUT, PB_IN, PB_OUT

Commit message: forgot to connect the pull-ups to voltage...
Connections:
- removed net N$1: RN7A.2, RN7B.2, RN7C.2, RN7D.2, RN8A.2, RN8B.2, RN8C.2, RN8D.2
- removed net N$2: RN5A.2, RN5B.2, RN5C.2, RN5D.2, RN6A.2, RN6B.2, RN6C.2, RN6D.2
- removed net N$20: PA_IN.2, PA_OUT.2
- new net 5V: PA_IN.2, PA_OUT.2, RN5A.2, RN5B.2, RN5C.2, RN5D.2, RN6A.2, RN6B.2, RN6C.2, RN6D.2, RN7A.2, RN7B.2, RN7C.2, RN7D.2, RN8A.2, RN8B.2, RN8C.2, RN8D.2
