File: pca9535bo.sch (EAGLE design)
At the start: 9 parts, among them IC1 PCA9535D, J1 0R, J2 0R, J3 0R

Commit message: the values need to be moved to the names layer to be seen...
Parts:
- PU2: value 4.7k -> I2C 4.7k
Changed lines of the file:
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@@
 <?xml version="1.0" encoding="utf-8"?>
 <!DOCTYPE eagle SYSTEM "eagle.dtd">
-<eagle version="6.1">
+<eagle version="6.2">
 <drawing>
 <settings>
@@
 <part name="J2" library="resistor" deviceset="R-EU_" device="R0603" value="0R"/>
 <part name="J3" library="resistor" deviceset="R-EU_" device="R0603" value="0R"/>
-<part name="PU2" library="resistor-dil" deviceset="4R-N" device="CAY16" value="4.7k"/>
+<part name="PU2" library="resistor-dil" deviceset="4R-N" device="CAY16" value="I2C 4.7k"/>
 </parts>
 <sheets>
